File: 2350/hardware/MSX_PicoVerse_2350_1.4/MSX_PicoVerse_2350_1.4.kicad_pcb (KiCad board)
At the start: 4 copper layers, 101.2 x 66.1 mm, 104 parts, among them IC1 AP63200WU-7, J11 MSX Cartridge Edge Fingers, J2 ESP-01, J3 SWD, J4 Micro_SD_Card, J5 USB_C_Receptacle_USB2.0_16P, Q1 DMMT5401, Q2 SSM3J332R, U1 Core2350B, U2 UDA1334MOD

Commit message: Rewrite README around the v1.2 differences; refresh gerbers and title blocks
README: drop the rev1.3 diode narrative. Add a 'How this differs from the original v1.2' section split into mechanical (laid out to a moulded cartridge shell) and electrical (buck, ideal-diode ORing, bus series resistors, TVS, polyfuse) changes, plus a stackup section.

Gerbers: re-plotted after the silkscreen fix - obsolete USB POWER / INT POWER labels removed, SWD labels moved next to J3.

Ordering: the JLCPCB stackup is JLC04161H-3313 as the order page spells it, not -3313A. Note that this special stackup disables Economic PCB assembly, so this board goes through Standard.

Title blocks: schematic and board were still stamped rev 1.3 / rev 1.2 with stale comments. Both now read rev 1.4, dated 2026-09-23.
Routing:
- net GND: vias 381 -> 389
Other:
- board text removed: "INT POWER"
- board text removed: "USB POWER"
Changed lines of the file:
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@@
 	(title_block
 		(title "MSX PicoVerse 2350")
-		(date "2026-07-26")
-		(rev "1.2")
+		(date "2026-09-23")
+		(rev "1.4")
 		(company "The Retro Hacker")
-		(comment 1 "Board reconstructed from the 1.2 production Gerber X2 / drill data")
+		(comment 1 "rev 1.4 by ESLAB - 4L JLC04161H-3313 1.6mm / ENIG + gold fingers / USB 90ohm diff L1-L2")
 	)
 	(layers
@@
 		(descr "SMD RESISTOR - 0603")
 		(property "Reference" "R48"
-			(at -1.07 -0.99 90)
+			(at -1.31 -0.85 90)
 			(unlocked yes)
 			(layer "F.SilkS")
@@
 		(tags "Through hole angled pin header THT 1x03 2.54mm single row")
 		(property "Reference" "J3"
-			(at -2.365 -0.27 0)
+			(at 1.5 7.54 0)
 			(layer "F.SilkS")
 			(effects
@@
 		(layer "Edge.Cuts")
 	)
-	(gr_text "USB\nPOWER"
-		(at 11.41 -57.01 0)
-		(layer "F.SilkS")
-		(effects
-			(font
-				(size 1.2 1)
-				(thickness 0.2)
-			)
-			(justify bottom)
-		)
-	)
-	(gr_text "INT\nPOWER"
-		(at 17.27 -56.95 0)
-		(layer "F.SilkS")
-		(effects
-			(font
-				(size 1.2 1)
-				(thickness 0.2)
-			)
-			(justify bottom)
-		)
-	)
-	(gr_text "GND"
-		(at -20.43 -23.95 90)
+	(gr_text "SWDIO"
+		(at -14.8 -56.3 90)
 		(layer "F.SilkS")
 		(effects
@@
 	)
 	(gr_text "SWLCK"
-		(at -17.89 -23.04 90)
+		(at -12.1 -56 90)
 		(layer "F.SilkS")
 		(effects
@@
 		)
 	)
-	(gr_text "SWDIO"
-		(at -15.36 -23.19 90)
+	(gr_text "GND"
+		(at -9.5 -57 90)
 		(layer "F.SilkS")
 		(effects
@@
 	)
 	(gr_text "DBUG"
-		(at -18.52 -18.62 0)
+		(at -12.6 -51.5 0)
 		(layer "F.SilkS")
 		(effects
@@
 	)
 	(via
+		(at 23.3 -54)
+		(size 0.6)
+		(drill 0.3)
+		(layers "F.Cu" "B.Cu")
+		(net "GND")
+	)
+	(via
 		(at -35.09 -35.42)
 		(size 0.6)
@@
 	)
 	(via
+		(at 36.8 -53.7)
+		(size 0.6)
+		(drill 0.3)
+		(layers "F.Cu" "B.Cu")
+		(net "GND")
+	)
+	(via
 		(at -17.65 -25.97)
 		(size 0.6)
@@
 	)
 	(via
+		(at 21 -51)
+		(size 0.6)
+		(drill 0.3)
+		(layers "F.Cu" "B.Cu")
+		(net "GND")
+	)
+	(via
 		(at 27.13 -55.62)
 		(size 0.6)
@@
 	)
 	(via
+		(at 35.1 -51.3)
+		(size 0.6)
+		(drill 0.3)
+		(layers "F.Cu" "B.Cu")
+		(net "GND")
+	)
+	(via
 		(at -51 -39)
 		(size 0.6)
@@
 	)
 	(via
+		(at 18.4 -54.1)
+		(size 0.6)
+		(drill 0.3)
+		(layers "F.Cu" "B.Cu")
+		(net "GND")
+	)
+	(via
 		(at 36 -27)
 		(size 0.6)
@@
 	)
 	(via
+		(at 33.8 -53.9)
+		(size 0.6)
+		(drill 0.3)
+		(layers "F.Cu" "B.Cu")
+		(net "GND")
+	)
+	(via
 		(at 33 -15)
 		(size 0.6)
@@
 	)
 	(via
+		(at 24.3 -51.1)
+		(size 0.6)
+		(drill 0.3)
+		(layers "F.Cu" "B.Cu")
+		(net "GND")
+	)
+	(via
 		(at 20.54 -55.58)
 		(size 0.6)
@@
 	)
 	(via
+		(at 17.8 -49.5)
+		(size 0.6)
+		(drill 0.3)
+		(layers "F.Cu" "B.Cu")
+		(net "GND")
+	)
+	(via
 		(at -2.21 -58.4)
 		(size 0.6)
@@
 	)
 	(segment
-		(start 12.906701 -40.975)
-		(end 13.031701 -40.85)
+		(start 23.47 -41.53)
+		(end 23.5 -41.56)
 		(width 0.25)
 		(layer "F.Cu")
@@
 	)
 	(segment
-		(start 8.45 -41.17)
-		(end 8.645 -40.975)
+		(start 13.031701 -40.85)
+		(end 22 -40.85)
 		(width 0.25)
 		(layer "F.Cu")
@@
 	)
 	(segment
-		(start 22 -40.85)
-		(end 22.68 -41.53)
+		(start 8.45 -41.17)
+		(end 8.52 -41.1)
 		(width 0.25)
 		(layer "F.Cu")
@@
 	)
 	(segment
-		(start 8.645 -40.975)
-		(end 12.906701 -40.975)
+		(start 23.5 -41.56)
+		(end 24 -41.56)
 		(width 0.25)
 		(layer "F.Cu")
@@
 	)
 	(segment
-		(start 23.5 -41.56)
-		(end 24 -41.56)
+		(start 8.52 -41.1)
+		(end 12.781701 -41.1)
 		(width 0.25)
 		(layer "F.Cu")
@@
 	)
 	(segment
-		(start 13.031701 -40.85)
-		(end 22 -40.85)
+		(start 22 -40.85)
+		(end 22.68 -41.53)
 		(width 0.25)
 		(layer "F.Cu")
@@
 	)
 	(segment
-		(start 23.47 -41.53)
-		(end 23.5 -41.56)
+		(start 12.781701 -41.1)
+		(end 13.031701 -40.85)
 		(width 0.25)
 		(layer "F.Cu")
@@
 		(layer "F.Cu")
 		(hatch none 0.1)
-		(priority 30082)
+		(priority 30107)
 		(attr
 			(teardrop
@@
 		(polygon
 			(pts
-				(xy -7.052051 -49.442565) (xy -7.047969 -50.042551) (xy -7.474693 -50.144955) (xy -7.851 -49.748007)
-				(xy -7.474693 -49.351045)
+				(xy -8.654286 -50.036425) (xy -8.645629 -49.436488) (xy -8.225307 -49.351045) (xy -7.849 -49.748014)
+				(xy -8.22887 -50.142574)
 			)
 		)
@@
 		(layer "F.Cu")
 		(hatch none 0.1)
-		(priority 30107)
+		(priority 30082)
 		(attr
 			(teardrop
@@
 		(polygon
 			(pts
-				(xy -8.654286 -50.036425) (xy -8.645629 -49.436488) (xy -8.225307 -49.351045) (xy -7.849 -49.748014)
-				(xy -8.22887 -50.142574)
+				(xy -7.052051 -49.442565) (xy -7.047969 -50.042551) (xy -7.474693 -50.144955) (xy -7.851 -49.748007)
+				(xy -7.474693 -49.351045)
 			)
 		)
@@
 		(layer "F.Cu")
 		(hatch none 0.1)
-		(priority 30077)
+		(priority 30078)
 		(attr
 			(teardrop
@@
 		(polygon
 			(pts
-				(xy 4.775 -53.15) (xy 5.025 -53.15) (xy 5.25 -53.5) (xy 4.9 -54.301) (xy 4.55 -53.5)
+				(xy 5.025 -55.45) (xy 4.775 -55.45) (xy 4.55 -55.1) (xy 4.9 -54.299) (xy 5.25 -55.1)
 			)
 		)
@@
 		(layer "F.Cu")
 		(hatch none 0.1)
-		(priority 30078)
+		(priority 30077)
 		(attr
 			(teardrop
@@
 		(polygon
 			(pts
-				(xy 5.025 -55.45) (xy 4.775 -55.45) (xy 4.55 -55.1) (xy 4.9 -54.299) (xy 5.25 -55.1)
+				(xy 4.775 -53.15) (xy 5.025 -53.15) (xy 5.25 -53.5) (xy 4.9 -54.301) (xy 4.55 -53.5)
 			)
 		)
@@
 	)
 	(zone
-		(net "/ESP01_UART_TX")
+		(net "+3V3")
 		(layer "F.Cu")
 		(hatch none 0.1)
-		(priority 30069)
+		(priority 30097)
 		(attr
 			(teardrop
@@
 		(polygon
 			(pts
-				(xy 22.113333 -41.14011) (xy 22.29011 -40.963333) (xy 22.68 -41.405) (xy 22.920242 -41.084205) (xy 23.504611 -41.53)
-				(xy 22.838559 -41.913548) (xy 22.68 -41.655) (xy 22.591612 -41.618388)
+				(xy -5.57 -49.428) (xy -5.57 -50.028) (xy -5.994693 -50.124955) (xy -6.371 -49.728) (xy -5.994693 -49.331045)
 			)
 		)
@@
 	)
 	(zone
-		(net "+3V3")
+		(net "/SPI_MOSI")
 		(layer "F.Cu")
 		(hatch none 0.1)
-		(priority 30097)
+		(priority 30079)
 		(attr
 			(teardrop
@@
 		(polygon
 			(pts
-				(xy -5.57 -49.428) (xy -5.57 -50.028) (xy -5.994693 -50.124955) (xy -6.371 -49.728) (xy -5.994693 -49.331045)
+				(xy 0.375 -53.15) (xy 0.625 -53.15) (xy 0.85 -53.5) (xy 0.5 -54.301) (xy 0.15 -53.5)
 			)
 		)
 	)
 	(zone
-		(net "/SPI_MOSI")
+		(net "Net-(U1-GP00)")
 		(layer "F.Cu")
 		(hatch none 0.1)
-		(priority 30079)
+		(priority 30177)
 		(attr
 			(teardrop
@@
 		(polygon
 			(pts
-				(xy 0.375 -53.15) (xy 0.625 -53.15) (xy 0.85 -53.5) (xy 0.5 -54.301) (xy 0.15 -53.5)
+				(xy -3.995 -14.762) (xy -4.245 -14.762) (xy -4.516955 -14.337307) (xy -4.12 -13.961) (xy -3.723045 -14.337307)
 			)
 		)
 	)
 	(zone
-		(net "Net-(U1-GP00)")
+		(net "+5V")
 		(layer "F.Cu")
 		(hatch none 0.1)
-		(priority 30177)
+		(priority 30062)
 		(attr
 			(teardrop
@@
 		(polygon
 			(pts
-				(xy -3.995 -14.762) (xy -4.245 -14.762) (xy -4.516955 -14.337307) (xy -4.12 -13.961) (xy -3.723045 -14.337307)
+				(xy -31.816 -37.362) (xy -31.816 -36.762) (xy -31.216 -36.462) (xy -30.615 -37.062) (xy -31.216 -37.65)
 			)
 		)
 	)
 	(zone
-		(net "+5V")
+		(net "/ESP01_UART_TX")
 		(layer "F.Cu")
 		(hatch none 0.1)
-		(priority 30062)
+		(priority 30069)
 		(attr
 			(teardrop
@@
 		(polygon
 			(pts
-				(xy -31.816 -37.362) (xy -31.816 -36.762) (xy -31.216 -36.462) (xy -30.615 -37.062) (xy -31.216 -37.65)
+				(xy 22.113333 -41.14011) (xy 22.29011 -40.963333) (xy 22.68 -41.405) (xy 22.920242 -41.084205) (xy 23.504611 -41.53)
+				(xy 22.838559 -41.913548) (xy 22.68 -41.655) (xy 22.591612 -41.618388)
 			)
 		)
